File: kicad/GradCapWiring.sch (KiCad schematic (older format))
At the start: 10 parts

Commit message: schematic update
Connections:
- net at Z?.~ (GND): now also A?.~ (VIN)
- net at A?.~ (VIN): no longer Z?.~ (GND)
- new net: A?.~ (VIN), J?.~ (Vout), J?.~ (Vout), Z?.~ (GND)
- now unconnected: A?.~ (VIN)
Other:
- note added: "Grad Cap"
Changed lines of the file:
@@
 	1    0    0    -1
 $EndComp
+Text Notes 8150 3000 0    197  ~ 39
+Grad Cap
 $EndSCHEMATC
